Commit message: working environment with moving robot

File: src/my_robot_description/urdf/my_robot.urdf.xacro (robot description, xacro)
@@ -1,4 +1,6 @@
 <?xml version="1.0"?>
-<robot name="my_robot">
+<robot name="my_robot" xmlns:xacro="http://www.ros.org/wiki/xacro">
+  <xacro:arg name="controller_config_file" default=""/>
+  <xacro:property name="controller_config_file" value="$(arg controller_config_file)"/>
   <link name="base_footprint"/>
   <joint name="base_joint" type="fixed">
@@ -133,10 +135,27 @@
   <gazebo reference="left_wheel_link">
     <material>Gazebo/Black</material>
+    <mu1>1.0</mu1>
+    <mu2>1.0</mu2>
+    <kp>1000000.0</kp>
+    <kd>100.0</kd>
+    <minDepth>0.001</minDepth>
+    <maxVel>1.0</maxVel>
   </gazebo>
   <gazebo reference="right_wheel_link">
     <material>Gazebo/Black</material>
+    <mu1>1.0</mu1>
+    <mu2>1.0</mu2>
+    <kp>1000000.0</kp>
+    <kd>100.0</kd>
+    <minDepth>0.001</minDepth>
+    <maxVel>1.0</maxVel>
   </gazebo>
   <gazebo reference="caster_wheel_link">
     <material>Gazebo/Grey</material>
+    <mu1>0.0</mu1>
+    <mu2>0.0</mu2>
+    <kp>1000000.0</kp>
+    <kd>100.0</kd>
+    <minDepth>0.001</minDepth>
   </gazebo>
   <gazebo reference="camera_link">
@@ -196,3 +215,8 @@
     </joint>
   </ros2_control>
+  <gazebo>
+    <plugin filename="libgazebo_ros2_control.so" name="gazebo_ros2_control">
+      <parameters>$(find my_robot_description)/config/my_robot_controllers.yaml</parameters>
+    </plugin>
+  </gazebo>
 </robot>
